Commit message: working urdf model

File: src/owi/model/owi.xacro (robot description, xacro)
@@ -1,44 +1,56 @@
 <?xml version="1.0" ?>
 <robot name="owi" xmlns:xacro="http://www.ros.org/wiki/xacro">
-  <xacro:property name="common_thickness" value="0.03" />
-  <!-- Macro to generate pure radial link for revolute joint -->
-  <xacro:macro name="radial_link" params="name length">
+  <xacro:property name="w" value="0.03" />
+  <!-- Macro to generate a link for manipulator, using reference frame of previous joint -->
+  <xacro:macro name="alink" params="name radial=0 axial=0">
     <link name="${name}">
+      <!-- elbow -->
       <visual>
         <geometry>
-          <box size="${length-common_thickness} ${common_thickness} ${common_thickness}" />
-        </geometry>
-        <origin rpy="0 0 0" xyz="${length/2} 0 0" />
-      </visual>
-      <visual>
-        <geometry>
-          <cylinder length="${common_thickness}" radius="${common_thickness/2}" />
+          <cylinder length="${w}" radius="${w/2}" />
         </geometry>
         <origin rpy="0 0 0" xyz="0 0 0" />
       </visual>
-    </link>
-  </xacro:macro>
-  <!-- Macro to generate a pure axial_link -->
-  <xacro:macro name="axial_link" params="name length">
-    <link name="${name}">
+      <!-- axial -->
       <visual>
         <geometry>
-          <cylinder length="${length}" radius = "${common_thickness/2}" />
+          <box size="${w} ${w} ${axial}" />
         </geometry>
-        <origin rpy="0 0 0" xyz="0 0 ${length/2}" />
+        <origin rpy="0 0 0" xyz="0 0 ${axial/2}" />
+      </visual>
+      <!-- radial -->
+      <visual>
+        <geometry>
+          <box size="${radial} ${w} ${w}" />
+        </geometry>
+        <origin rpy="0 0 0" xyz="${radial/2} 0 ${axial}" />
       </visual>
     </link>
   </xacro:macro>
-  <!-- Macro to generate revolute joint on D-H convention -->
-  <!-- Assume position theta* = 0, radial and twist can use parent x axis -->
+  <!-- Macro to generate a joint on D-H convention, using reference frame of previous joint -->
+  <!-- Assume position theta* = 0, radial and twist are along/around parent x axis -->
   <!-- Use degree for angle -->
-  <xacro:macro name="revolute_joint" params="parent child radial axial twist lo_limit hi_limit">
-    <joint name="${parent}_${child}" type="revolute">
+  <xacro:macro name="ajoint" params="type parent child radial=0 axial=0 twist=0 lo_limit=-180 hi_limit=180 effort=100 velocity=1">
+    <joint name="${parent}_${child}" type="${type}">
       <parent link="${parent}" />
       <child link="${child}" />
       <axis xyz="0 0 1" />
       <origin rpy="${pi*twist/180} 0 0" xyz="${radial} 0 ${axial}" />
-      <limit effort="100" lower="${pi*lo_limit/180}" upper="${pi*hi_limit/180}" velocity="1" />
+      <!-- revolute joint -->
+      <xacro:if value="${type == 'revolute'}">
+        <limit effort="${effort}" lower="${pi*lo_limit/180}" upper="${pi*hi_limit/180}" velocity="${velocity}" />
+      </xacro:if>
+      <!-- prismatic joint -->
+      <xacro:if value="${type == 'prismatic'}">
+        <limit effort="${effort}" lower="${lo_limit}" upper="${hi_limit}" velocity="${velocity}" />
+      </xacro:if>
     </joint>
+  </xacro:macro>
+  <!-- Macro to generate a joint and link from previous joint, using reference frame of previous joint -->
+  <!-- Assume position theta* = 0, radial and twist can use previous joint x axis -->
+  <!-- Use degree for angle -->
+  <xacro:macro name="linked_joint" params="type parent child radial=0 axial=0 twist=0 lo_limit hi_limit">
+    <xacro:alink name="${parent}" radial="${radial}" axial="${axial}" />
+    <xacro:ajoint type="${type}" parent="${parent}" child="${child}" radial="${radial}" axial="${axial}" twist="${twist}" lo_limit="${lo_limit}" hi_limit="${hi_limit}" />
   </xacro:macro>
   <!-- robot model  -->
@@ -52,22 +64,21 @@
     <visual>
       <geometry>
-        <cylinder length="${common_thickness}" radius="${common_thickness}" />
+        <cylinder length="${w}" radius="${w}" />
       </geometry>
-      <origin rpy="0 0 0" xyz="0 0 ${common_thickness/2}" />
+      <origin rpy="0 0 0" xyz="0 0 ${w/2}" />
     </visual>
     <visual>
       <geometry>
-        <box size="0.12 0.06 ${common_thickness}" />
+        <box size="0.12 0.06 ${w}" />
       </geometry>
-      <origin rpy="0 0 0" xyz="-0.06 0 ${common_thickness/2}" />
+      <origin rpy="0 0 0" xyz="-0.06 0 ${w/2}" />
     </visual>
   </link>
-  <xacro:revolute_joint parent="base_link" child="link1" radial="0" axial="${1.5*common_thickness}" twist="0" lo_limit="-90" hi_limit="90" />
-  <xacro:axial_link name="link1" length="0" />
-  <xacro:revolute_joint parent="link1" child="link2" radial="0" axial="0" twist="90" lo_limit="0" hi_limit="180" />
-  <xacro:radial_link name="link2" length="0.085" />
-  <xacro:revolute_joint parent="link2" child="link3" radial="0.085" axial="0" twist="0" lo_limit="-135" hi_limit="135" />
-  <xacro:radial_link name="link3" length="0.115" />
-  <xacro:revolute_joint parent="link3" child="link4" radial="0.115" axial="0" twist="0" lo_limit="-60" hi_limit="60" />
-  <xacro:radial_link name="link4" length="0.05" />
+  <xacro:ajoint type="revolute" parent="base_link" child="link1" axial="${1.5*w}" lo_limit="-90" hi_limit="90" />
+  <xacro:linked_joint type="revolute" parent="link1" child="link2" twist="90" lo_limit="0" hi_limit="180" />
+  <xacro:linked_joint type="revolute" parent="link2" child="link3" radial="0.085" lo_limit="-135" hi_limit="135" />
+  <xacro:linked_joint type="revolute" parent="link3" child="link4" radial="0.115" lo_limit="-60" hi_limit="60" />
+  <xacro:linked_joint type="revolute" parent="link4" child="gripper" radial="0.05" lo_limit="-60" hi_limit="60" />
+  <link name="gripper">
+  </link>
 </robot>

Commit message: updated urdf with collision

File: src/owi/model/owi.xacro (robot description, xacro)
@@ -1,7 +1,6 @@
 <?xml version="1.0" ?>
 <robot name="owi" xmlns:xacro="http://www.ros.org/wiki/xacro">
-  <xacro:property name="w" value="0.03" />
   <!-- Macro to generate a link for manipulator, using reference frame of previous joint -->
-  <xacro:macro name="alink" params="name radial=0 axial=0">
+  <xacro:macro name="alink" params="name radial=0 axial=0 w=0.03" >
     <link name="${name}">
       <!-- elbow -->
@@ -12,18 +11,36 @@
         <origin rpy="0 0 0" xyz="0 0 0" />
       </visual>
+      <collision>
+        <geometry>
+          <cylinder length="${w}" radius="${w/2}" />
+        </geometry>
+        <origin rpy="0 0 0" xyz="0 0 0" />
+      </collision>
       <!-- axial -->
       <visual>
         <geometry>
-          <box size="${w} ${w} ${axial}" />
+          <box size="${w/2} ${w/2} ${axial}" />
         </geometry>
         <origin rpy="0 0 0" xyz="0 0 ${axial/2}" />
       </visual>
+      <collision>
+        <geometry>
+          <box size="${w/2} ${w/2} ${axial/2}" />
+        </geometry>
+        <origin rpy="0 0 0" xyz="0 0 ${axial/2}" />
+      </collision>
       <!-- radial -->
       <visual>
         <geometry>
-          <box size="${radial} ${w} ${w}" />
+          <box size="${radial/2} ${w/2} ${w/2}" />
         </geometry>
         <origin rpy="0 0 0" xyz="${radial/2} 0 ${axial}" />
       </visual>
+      <collision>
+        <geometry>
+          <box size="${radial/2} ${w/2} ${w/2}" />
+        </geometry>
+        <origin rpy="0 0 0" xyz="${radial/2} 0 ${axial}" />
+      </collision>
     </link>
   </xacro:macro>
@@ -47,11 +64,4 @@
     </joint>
   </xacro:macro>
-  <!-- Macro to generate a joint and link from previous joint, using reference frame of previous joint -->
-  <!-- Assume position theta* = 0, radial and twist can use previous joint x axis -->
-  <!-- Use degree for angle -->
-  <xacro:macro name="linked_joint" params="type parent child radial=0 axial=0 twist=0 lo_limit hi_limit">
-    <xacro:alink name="${parent}" radial="${radial}" axial="${axial}" />
-    <xacro:ajoint type="${type}" parent="${parent}" child="${child}" radial="${radial}" axial="${axial}" twist="${twist}" lo_limit="${lo_limit}" hi_limit="${hi_limit}" />
-  </xacro:macro>
   <!-- robot model  -->
   <link name="world" />
@@ -64,21 +74,38 @@
     <visual>
       <geometry>
-        <cylinder length="${w}" radius="${w}" />
+        <cylinder length="0.05" radius="0.05" />
       </geometry>
-      <origin rpy="0 0 0" xyz="0 0 ${w/2}" />
+      <origin rpy="0 0 0" xyz="0 0 0.025" />
     </visual>
     <visual>
       <geometry>
-        <box size="0.12 0.06 ${w}" />
+        <box size="0.15 0.08 0.05" />
       </geometry>
-      <origin rpy="0 0 0" xyz="-0.06 0 ${w/2}" />
+      <origin rpy="0 0 0" xyz="-0.1 0 0.025" />
     </visual>
+    <collision>
+      <geometry>
+        <cylinder length="0.05" radius="0.05" />
+      </geometry>
+      <origin rpy="0 0 0" xyz="0 0 0.025" />
+    </collision>
+    <collision>
+      <geometry>
+        <box size="0.15 0.08 0.05" />
+      </geometry>
+      <origin rpy="0 0 0" xyz="-0.1 0 0.025" />
+    </collision>
   </link>
-  <xacro:ajoint type="revolute" parent="base_link" child="link1" axial="${1.5*w}" lo_limit="-90" hi_limit="90" />
-  <xacro:linked_joint type="revolute" parent="link1" child="link2" twist="90" lo_limit="0" hi_limit="180" />
-  <xacro:linked_joint type="revolute" parent="link2" child="link3" radial="0.085" lo_limit="-135" hi_limit="135" />
-  <xacro:linked_joint type="revolute" parent="link3" child="link4" radial="0.115" lo_limit="-60" hi_limit="60" />
-  <xacro:linked_joint type="revolute" parent="link4" child="gripper" radial="0.05" lo_limit="-60" hi_limit="60" />
-  <link name="gripper">
-  </link>
+  <xacro:ajoint type="revolute" parent="base_link" child="link1" axial="0.065" lo_limit="-90" hi_limit="90" />
+  <link name="link1" />
+  <xacro:ajoint type="revolute" parent="link1" child="link2" twist="90" lo_limit="0" hi_limit="180" />
+  <xacro:alink name="link2" radial="0.085" />
+  <xacro:ajoint type="revolute" parent="link2" child="link3" radial="0.085" lo_limit="-135" hi_limit="135" />
+  <xacro:alink name="link3" radial="0.115" />
+  <xacro:ajoint type="revolute" parent="link3" child="link4" radial="0.115" lo_limit="-60" hi_limit="60" />
+  <xacro:alink name="link4" radial="0.06" />
+  <xacro:ajoint type="revolute" parent="link4" child="r_gripper" twist="90" radial="0.06" axial="0.005" lo_limit="0" hi_limit="90" />
+  <xacro:ajoint type="revolute" parent="link4" child="l_gripper" twist="-90" radial="0.06" axial="-0.005" lo_limit="0" hi_limit="90" />
+  <xacro:alink name="l_gripper" radial="0.03" w="0.01" />
+  <xacro:alink name="r_gripper" radial="0.03" w="0.01" />
 </robot>

Commit message: working on joint_state_publisher

File: src/owi/model/owi.xacro (robot description, xacro)
@@ -48,6 +48,6 @@
   <!-- Assume position theta* = 0, radial and twist are along/around parent x axis -->
   <!-- Use degree for angle -->
-  <xacro:macro name="ajoint" params="type parent child radial=0 axial=0 twist=0 lo_limit=-180 hi_limit=180 effort=100 velocity=1">
-    <joint name="${parent}_${child}" type="${type}">
+  <xacro:macro name="ajoint" params="type parent child radial=0 axial=0 twist=0 lo_limit=-180 hi_limit=180 effort=100 velocity=1 mimic=none">
+    <joint name="$joint${child}" type="${type}">
       <parent link="${parent}" />
       <child link="${child}" />
@@ -62,14 +62,18 @@
         <limit effort="${effort}" lower="${lo_limit}" upper="${hi_limit}" velocity="${velocity}" />
       </xacro:if>
+      <!-- mimic joint -->
+      <xacro:if value="${mimic != 'none'}">
+        <mimic joint="${mimic}" />>
+      </xacro:if>
     </joint>
   </xacro:macro>
   <!-- robot model  -->
   <link name="world" />
-  <joint name="world_to_base" type="fixed">
+  <joint name="worldBase" type="fixed">
     <parent link="world" />
-    <child link="base_link" />
+    <child link="baselink" />
     <origin rpy="0 0 0" xyz="0 0 0" />
   </joint>
-  <link name="base_link">
+  <link name="baselink">
     <visual>
       <geometry>
@@ -97,15 +101,15 @@
     </collision>
   </link>
-  <xacro:ajoint type="revolute" parent="base_link" child="link1" axial="0.065" lo_limit="-90" hi_limit="90" />
-  <link name="link1" />
-  <xacro:ajoint type="revolute" parent="link1" child="link2" twist="90" lo_limit="0" hi_limit="180" />
-  <xacro:alink name="link2" radial="0.085" />
-  <xacro:ajoint type="revolute" parent="link2" child="link3" radial="0.085" lo_limit="-135" hi_limit="135" />
-  <xacro:alink name="link3" radial="0.115" />
-  <xacro:ajoint type="revolute" parent="link3" child="link4" radial="0.115" lo_limit="-60" hi_limit="60" />
-  <xacro:alink name="link4" radial="0.06" />
-  <xacro:ajoint type="revolute" parent="link4" child="r_gripper" twist="90" radial="0.06" axial="0.005" lo_limit="0" hi_limit="90" />
-  <xacro:ajoint type="revolute" parent="link4" child="l_gripper" twist="-90" radial="0.06" axial="-0.005" lo_limit="0" hi_limit="90" />
-  <xacro:alink name="l_gripper" radial="0.03" w="0.01" />
-  <xacro:alink name="r_gripper" radial="0.03" w="0.01" />
+  <xacro:ajoint type="revolute" parent="baselink" child="Link1" axial="0.065" lo_limit="-90" hi_limit="90" />
+  <link name="Link1" />
+  <xacro:ajoint type="revolute" parent="Link1" child="Link2" twist="90" lo_limit="0" hi_limit="180" />
+  <xacro:alink name="Link2" radial="0.085" />
+  <xacro:ajoint type="revolute" parent="Link2" child="Link3" radial="0.085" lo_limit="-135" hi_limit="135" />
+  <xacro:alink name="Link3" radial="0.115" />
+  <xacro:ajoint type="revolute" parent="Link3" child="Link4" radial="0.115" lo_limit="-60" hi_limit="60" />
+  <xacro:alink name="Link4" radial="0.06" />
+  <xacro:ajoint type="revolute" parent="Link4" child="Rgripper" twist="90" radial="0.06" axial="0.005" lo_limit="0" hi_limit="90" />
+  <!-- <xacro:ajoint type="revolute" parent="Link4" child="Lgripper" twist="-90" radial="0.06" axial="-0.005" lo_limit="0" hi_limit="90" mimic="Link4Rgripper" /> -->
+  <xacro:alink name="Rgripper" radial="0.03" w="0.01" />
+  <!-- <xacro:alink name="Lgripper" radial="0.03" w="0.01" /> -->
 </robot>

Commit message: fixed typo causing seemingly mimictag problem

File: src/owi/model/owi.xacro (robot description, xacro)
@@ -49,5 +49,5 @@
   <!-- Use degree for angle -->
   <xacro:macro name="ajoint" params="type parent child radial=0 axial=0 twist=0 lo_limit=-180 hi_limit=180 effort=100 velocity=1 mimic=none">
-    <joint name="$joint${child}" type="${type}">
+    <joint name="joint_${child}" type="${type}">
       <parent link="${parent}" />
       <child link="${child}" />
@@ -64,5 +64,5 @@
       <!-- mimic joint -->
       <xacro:if value="${mimic != 'none'}">
-        <mimic joint="${mimic}" />>
+        <mimic joint="${mimic}" />
       </xacro:if>
     </joint>
@@ -70,10 +70,10 @@
   <!-- robot model  -->
   <link name="world" />
-  <joint name="worldBase" type="fixed">
+  <joint name="jointBase" type="fixed">
     <parent link="world" />
-    <child link="baselink" />
+    <child link="base_link" />
     <origin rpy="0 0 0" xyz="0 0 0" />
   </joint>
-  <link name="baselink">
+  <link name="base_link">
     <visual>
       <geometry>
@@ -101,5 +101,5 @@
     </collision>
   </link>
-  <xacro:ajoint type="revolute" parent="baselink" child="Link1" axial="0.065" lo_limit="-90" hi_limit="90" />
+  <xacro:ajoint type="revolute" parent="base_link" child="Link1" axial="0.065" lo_limit="-90" hi_limit="90" />
   <link name="Link1" />
   <xacro:ajoint type="revolute" parent="Link1" child="Link2" twist="90" lo_limit="0" hi_limit="180" />
@@ -110,6 +110,6 @@
   <xacro:alink name="Link4" radial="0.06" />
   <xacro:ajoint type="revolute" parent="Link4" child="Rgripper" twist="90" radial="0.06" axial="0.005" lo_limit="0" hi_limit="90" />
-  <!-- <xacro:ajoint type="revolute" parent="Link4" child="Lgripper" twist="-90" radial="0.06" axial="-0.005" lo_limit="0" hi_limit="90" mimic="Link4Rgripper" /> -->
+  <xacro:ajoint type="revolute" parent="Link4" child="Lgripper" twist="-90" radial="0.06" axial="-0.005" lo_limit="0" hi_limit="90" mimic="joint_Rgripper" />
   <xacro:alink name="Rgripper" radial="0.03" w="0.01" />
-  <!-- <xacro:alink name="Lgripper" radial="0.03" w="0.01" /> -->
+  <xacro:alink name="Lgripper" radial="0.03" w="0.01" />
 </robot>

Commit message: fixed deg to rad issue'

File: src/owi/model/owi.xacro (robot description, xacro)
@@ -49,5 +49,5 @@
   <!-- Use degree for angle -->
   <xacro:macro name="ajoint" params="type parent child radial=0 axial=0 twist=0 lo_limit=-180 hi_limit=180 effort=100 velocity=1 mimic=none">
-    <joint name="$joint${child}" type="${type}">
+    <joint name="joint${child}" type="${type}">
       <parent link="${parent}" />
       <child link="${child}" />
@@ -64,15 +64,9 @@
       <!-- mimic joint -->
       <xacro:if value="${mimic != 'none'}">
-        <mimic joint="${mimic}" />>
+        <mimic joint="${mimic}" />
       </xacro:if>
     </joint>
   </xacro:macro>
   <!-- robot model  -->
-  <link name="world" />
-  <joint name="worldBase" type="fixed">
-    <parent link="world" />
-    <child link="baselink" />
-    <origin rpy="0 0 0" xyz="0 0 0" />
-  </joint>
   <link name="baselink">
     <visual>
@@ -110,6 +104,6 @@
   <xacro:alink name="Link4" radial="0.06" />
   <xacro:ajoint type="revolute" parent="Link4" child="Rgripper" twist="90" radial="0.06" axial="0.005" lo_limit="0" hi_limit="90" />
-  <!-- <xacro:ajoint type="revolute" parent="Link4" child="Lgripper" twist="-90" radial="0.06" axial="-0.005" lo_limit="0" hi_limit="90" mimic="Link4Rgripper" /> -->
+  <xacro:ajoint type="revolute" parent="Link4" child="Lgripper" twist="-90" radial="0.06" axial="-0.005" lo_limit="0" hi_limit="90" mimic="jointRgripper" />
   <xacro:alink name="Rgripper" radial="0.03" w="0.01" />
-  <!-- <xacro:alink name="Lgripper" radial="0.03" w="0.01" /> -->
+  <xacro:alink name="Lgripper" radial="0.03" w="0.01" />
 </robot>

Commit message: consolidate rviz.launch

File: src/owi/model/owi.xacro (robot description, xacro)
@@ -69,5 +69,5 @@
   </xacro:macro>
   <!-- robot model  -->
-  <link name="baselink">
+  <link name="base_link">
     <visual>
       <geometry>

Commit message: added moveit package

File: src/owi/model/owi.xacro (robot description, xacro)
@@ -43,4 +43,8 @@
         <origin rpy="0 0 0" xyz="${radial/2} 0 ${axial}" />
       </collision>
+      <intnertial>
+        <mass value="0.1"/>
+        <inertia ixx="0.033" iyy="0.033" izz="0.033" ixy="0.0" ixz="0.0" iyz="0.0"/>
+      </intnertial>
     </link>
   </xacro:macro>
@@ -84,5 +88,5 @@
     <collision>
       <geometry>
-        <cylinder length="0.05" radius="0.05" />
+        <cylinder length="0.04" radius="0.05" />
       </geometry>
       <origin rpy="0 0 0" xyz="0 0 0.025" />
@@ -94,4 +98,8 @@
       <origin rpy="0 0 0" xyz="-0.1 0 0.025" />
     </collision>
+    <intnertial>
+      <mass value="0.3"/>
+      <inertia ixx="0.1" iyy="0.1" izz="0.1" ixy="0.0" ixz="0.0" iyz="0.0"/>
+    </intnertial>
   </link>
   <xacro:ajoint type="revolute" parent="base_link" child="Link1" axial="0.065" lo_limit="-90" hi_limit="90" />
@@ -103,6 +111,21 @@
   <xacro:ajoint type="revolute" parent="Link3" child="Link4" radial="0.115" lo_limit="-60" hi_limit="60" />
   <xacro:alink name="Link4" radial="0.06" />
-  <xacro:ajoint type="revolute" parent="Link4" child="Rgripper" twist="90" radial="0.06" axial="0.005" lo_limit="0" hi_limit="90" />
-  <xacro:ajoint type="revolute" parent="Link4" child="Lgripper" twist="-90" radial="0.06" axial="-0.005" lo_limit="0" hi_limit="90" mimic="jointRgripper" />
+  <joint name="dummy1" type="revolute">
+    <parent link="Link4" />
+    <child link="grip_base" />
+    <axis xyz="0 0 1" />
+    <origin rpy="${0.5*pi} 0 0" xyz="0.06 0 0" />
+    <limit effort="100" velocity="1" lower="-10" upper="10" />
+  </joint>
+  <link name="grip_base">
+    <visual>
+      <geometry>
+        <box size="0 0 0" />
+      </geometry>
+      <origin rpy="0 0 0" xyz="0 0 0" />
+    </visual>
+  </link>
+  <xacro:ajoint type="revolute" parent="Link4" child="Rgripper" twist="90" radial="0.06" axial="0.006" lo_limit="0" hi_limit="90" />
+  <xacro:ajoint type="revolute" parent="Link4" child="Lgripper" twist="-90" radial="0.06" axial="-0.006" lo_limit="0" hi_limit="90" mimic="jointRgripper" />
   <xacro:alink name="Rgripper" radial="0.03" w="0.01" />
   <xacro:alink name="Lgripper" radial="0.03" w="0.01" />
