Commit message: set ik to position only

File: src/owi_moveit/config/owi.xacro (robot description, xacro)
@@ -33,5 +33,5 @@
       <visual>
         <geometry>
-          <box size="${radial/2} ${w/2} ${w/2}" />
+          <box size="${radial} ${w/2} ${w/2}" />
         </geometry>
         <origin rpy="0 0 0" xyz="${radial/2} 0 ${axial}" />
@@ -39,5 +39,5 @@
       <collision>
         <geometry>
-          <box size="${radial/2} ${w/2} ${w/2}" />
+          <box size="${radial} ${w/2} ${w/2}" />
         </geometry>
         <origin rpy="0 0 0" xyz="${radial/2} 0 ${axial}" />
@@ -111,12 +111,12 @@
   <xacro:ajoint type="revolute" parent="Link3" child="Link4" radial="0.115" lo_limit="-60" hi_limit="60" />
   <xacro:alink name="Link4" radial="0.06" />
-  <joint name="dummy1" type="revolute">
+  <joint name="dummy_joint" type="revolute">
     <parent link="Link4" />
-    <child link="grip_base" />
+    <child link="dummy_eef" />
     <axis xyz="0 0 1" />
     <origin rpy="${0.5*pi} 0 0" xyz="0.06 0 0" />
     <limit effort="100" velocity="1" lower="-10" upper="10" />
   </joint>
-  <link name="grip_base">
+  <link name="dummy_eef">
     <visual>
       <geometry>

Commit message: robot following fake execution

File: src/owi_moveit/config/owi.xacro (robot description, xacro)
@@ -94,7 +94,7 @@
     <collision>
       <geometry>
-        <box size="0.15 0.08 0.05" />
+        <box size="0.15 0.08 0.08" />
       </geometry>
-      <origin rpy="0 0 0" xyz="-0.1 0 0.025" />
+      <origin rpy="0 0 0" xyz="-0.1 0 0.04" />
     </collision>
     <intnertial>

Commit message: added kinect2 face detection

File: src/owi_moveit/config/owi.xacro (robot description, xacro)
@@ -103,4 +103,23 @@
     </intnertial>
   </link>
+  <joint name="camera_fixed" type="fixed">
+    <parent link="base_link" />
+    <child link="kinect2_link" />
+    <origin rpy="${-0.5*pi} 0 ${-0.25*pi}" xyz="-0.5 -0.5 0" />
+  </joint>
+  <link name="kinect2_link" />
+  <joint name="nose_pos" type="floating">
+    <parent link="kinect2_link" />
+    <child link="nose_link" />
+    <origin rpy="0 0 0" xyz="0 0 0" />
+  </joint>
+  <link name="nose_link">
+      <visual>
+      <geometry>
+        <sphere radius="0.03" />
+      </geometry>
+      <origin rpy="0 0 0" xyz="0 0 0" />
+    </visual>
+  </link>
   <xacro:ajoint type="revolute" parent="base_link" child="Link1" axial="0.065" lo_limit="-90" hi_limit="90" />
   <link name="Link1" />
@@ -118,12 +137,5 @@
     <limit effort="100" velocity="1" lower="-10" upper="10" />
   </joint>
-  <link name="dummy_eef">
-    <visual>
-      <geometry>
-        <box size="0 0 0" />
-      </geometry>
-      <origin rpy="0 0 0" xyz="0 0 0" />
-    </visual>
-  </link>
+  <link name="dummy_eef" />
   <xacro:ajoint type="revolute" parent="Link4" child="Rgripper" twist="90" radial="0.06" axial="0.006" lo_limit="0" hi_limit="90" />
   <xacro:ajoint type="revolute" parent="Link4" child="Lgripper" twist="-90" radial="0.06" axial="-0.006" lo_limit="0" hi_limit="90" mimic="jointRgripper" />

Commit message: Motion planning not reliable yet

File: src/owi_moveit/config/owi.xacro (robot description, xacro)
@@ -103,23 +103,4 @@
     </intnertial>
   </link>
-  <joint name="camera_fixed" type="fixed">
-    <parent link="base_link" />
-    <child link="kinect2_link" />
-    <origin rpy="${-0.5*pi} 0 ${-0.25*pi}" xyz="-0.5 -0.5 0" />
-  </joint>
-  <link name="kinect2_link" />
-  <joint name="nose_pos" type="floating">
-    <parent link="kinect2_link" />
-    <child link="nose_link" />
-    <origin rpy="0 0 0" xyz="0 0 0" />
-  </joint>
-  <link name="nose_link">
-      <visual>
-      <geometry>
-        <sphere radius="0.03" />
-      </geometry>
-      <origin rpy="0 0 0" xyz="0 0 0" />
-    </visual>
-  </link>
   <xacro:ajoint type="revolute" parent="base_link" child="Link1" axial="0.065" lo_limit="-90" hi_limit="90" />
   <link name="Link1" />
@@ -142,3 +123,31 @@
   <xacro:alink name="Rgripper" radial="0.03" w="0.01" />
   <xacro:alink name="Lgripper" radial="0.03" w="0.01" />
+  <!-- Kinect camera -->
+  <joint name="camera_fixed" type="fixed">
+    <parent link="base_link" />
+    <child link="kinect2_link" />
+    <origin rpy="${-0.4*pi} 0 ${-0.25*pi}" xyz="-0.3 -0.3 -0.1" />
+  </joint>
+  <link name="kinect2_link">
+    <visual>
+      <origin rpy="${-pi/2} 0 ${pi}" xyz="0.1 0 0" />
+      <geometry>
+        <mesh filename="package://owi_moveit/meshes/kinect.stl" scale="0.001 0.001 0.001" />
+      </geometry>
+    </visual>
+  </link>
+  <!-- Nose marker -->
+  <joint name="nose_pos" type="floating">
+    <parent link="kinect2_link" />
+    <child link="nose_link" />
+    <origin rpy="0 0 0" xyz="0 0 0" />
+  </joint>
+  <link name="nose_link">
+      <visual>
+      <geometry>
+        <sphere radius="0.02" />
+      </geometry>
+      <origin rpy="0 0 0" xyz="0 0 0" />
+    </visual>
+  </link>
 </robot>
